File: Matrix/.history/Matrix.kicad_sch (KiCad schematic)
At the start: 55 parts, among them J1 Conn_01x08, Q1 2N2219, Q10 2N2219, Q11 2N2219, Q12 2N2219, Q13 2N2219, Q14 2N2219, Q15 2N2219, Q16 2N2219, Q2 2N2219, Q3 2N2219, Q4 2N2219, Q5 2N2219, Q6 2N2219, Q7 2N2219, Q8 2N2219, Q9 2N2219, U1 74HC138

Commit message: Update Matrix.kicad_sch
Connections:
- net +5V: now also U1.4 (~{E0})
- net A1: now also U1.1 (A0)
- net A2: now also U1.2 (A1)
- net A3: now also U1.3 (A2)
- net GND: now also U1.5 (~{E1}), U1.6 (E2)

Commit message: Update Matrix.kicad_sch
Parts:
- added R25, R26, R27, R28, R29, R30, R31, R32, R33, R34, R35, R36, R37, R38, R39, R40, R41, R42, R43, R44, R45, R46, R47, R48, R49, R50, R51, R52, R53, R54, R55, R56, R57, R58, R59, R60, R61, R62, R63, R64, R65, R66, R67, R68, R69, R70, R71, R72, R73, R74, R75, R76, R77, R78, R79, R80, R81, R82, R83, R84, R85, R86, R87, R88: 100R, Resistor_SMD:R_0815_2038Metric, symbol Device:R
- added ROW1, ROW2, ROW3, ROW4, ROW5, ROW6, ROW7, ROW8: Conn_01x08, Connector_PinHeader_1.00mm:PinHeader_1x08_P1.00mm_Horizontal, symbol Connector_Generic:Conn_01x08
- added U2, U3, U4, U5, U6, U7, U8: 74HC574N, 74HC574N:DIP254P762X420-20, symbol 74HC574N:74HC574N
- added U9: 74HC574N, DIP254P762X420-20, symbol 74HC574N:74HC574N
- C1, C2, C3, C4, C5, C6, C7, C8, C9: footprint (none) -> Capacitor_SMD:C_0805_2012Metric
- C10: footprint (none) -> Capacitor_THT:CP_Axial_L10.0mm_D4.5mm_P15.00mm_Horizontal
- C11, C12: footprint (none) -> Capacitor_SMD:C_0805_2012Metric_Pad1.18x1.45mm_HandSolder
- J1: footprint (none) -> Connector_PinHeader_1.00mm:PinHeader_1x08_P1.00mm_Horizontal
- R1, R10, R11, R12, R13, R14, R15, R16, R17, R18, R2, R3, R4, R5, R6, R7, R8, R9: footprint (none) -> Resistor_SMD:R_0815_2038Metric_Pad1.20x4.05mm_HandSolder
- R19, R20, R21, R22, R23, R24: footprint (none) -> Resistor_SMD:R_0815_2038Metric
- U1: footprint (none) -> 74HC138D:SOIC127P600X175-16N
Connections:
- net D0: now also U2.2 (D0), U3.2 (D0), U4.2 (D0), U5.2 (D0), U6.2 (D0), U7.2 (D0), U8.2 (D0), U9.2 (D0)
- net D1: now also U2.3 (D1), U3.3 (D1), U4.3 (D1), U5.3 (D1), U6.3 (D1), U7.3 (D1), U8.3 (D1), U9.3 (D1)
- net D2: now also U2.4 (D2), U3.4 (D2), U4.4 (D2), U5.4 (D2), U6.4 (D2), U7.4 (D2), U8.4 (D2), U9.4 (D2)
- net D3: now also U2.5 (D3), U3.5 (D3), U4.5 (D3), U5.5 (D3), U6.5 (D3), U7.5 (D3), U8.5 (D3), U9.5 (D3)
- net D4: now also U2.6 (D4), U3.6 (D4), U4.6 (D4), U5.6 (D4), U6.6 (D4), U7.6 (D4), U8.6 (D4), U9.6 (D4)
- net D5: now also U2.7 (D5), U3.7 (D5), U4.7 (D5), U5.7 (D5), U6.7 (D5), U7.7 (D5), U8.7 (D5), U9.7 (D5)
- net D6: now also U2.8 (D6), U3.8 (D6), U4.8 (D6), U5.8 (D6), U6.8 (D6), U7.8 (D6), U8.8 (D6), U9.8 (D6)
- net D7: now also U2.9 (D7), U3.9 (D7), U4.9 (D7), U5.9 (D7), U6.9 (D7), U7.9 (D7), U8.9 (D7), U9.9 (D7)
- net GND: now also Q2.1 (E), Q3.1 (E), U2.10 (GND), U2.20 (VCC), U3.10 (GND), U3.20 (VCC), U4.10 (GND), U4.20 (VCC), U5.10 (GND), U5.20 (VCC), U6.10 (GND), U6.20 (VCC), U7.10 (GND), U7.20 (VCC), U8.10 (GND), U8.20 (VCC), U9.10 (GND), U9.20 (VCC)
- net OE: now also U2.1 (~{OE}), U3.1 (~{OE}), U4.1 (~{OE}), U5.1 (~{OE}), U6.1 (~{OE}), U7.1 (~{OE}), U8.1 (~{OE}), U9.1 (~{OE})
- net at U1.10 (~{Y5}): now also U7.11 (CP)
- net at U1.11 (~{Y4}): now also U6.11 (CP)
- net at U1.12 (~{Y3}): now also U5.11 (CP)
- net at U1.13 (~{Y2}): now also U4.11 (CP)
- net at U1.14 (~{Y1}): now also U3.11 (CP)
- net at U1.15 (~{Y0}): now also U2.11 (CP)
- net at U1.7 (~{Y7}): now also U9.11 (CP)
- net at U1.9 (~{Y6}): now also U8.11 (CP)
- new net: R65.1, U7.12 (Q7)
- new net: R65.2, ROW6.1 (Pin_1)
- new net: R71.1, U7.18 (Q1)
- new net: R71.2, ROW6.7 (Pin_7)
- new net: R28.1, U2.15 (Q4)
- new net: R28.2, ROW1.4 (Pin_4)
- new net: R30.1, U2.17 (Q2)
- new net: R30.2, ROW1.6 (Pin_6)
- new net: R70.1, U7.17 (Q2)
- new net: R70.2, ROW6.6 (Pin_6)
- new net: R25.1, U2.12 (Q7)
- new net: R26.1, U2.13 (Q6)
- new net: R27.1, U2.14 (Q5)
- new net: R29.1, U2.16 (Q3)
- new net: R31.1, U2.18 (Q1)
- new net: R32.1, U2.19 (Q0)
- new net: R81.1, U9.12 (Q7)
- new net: R81.2, ROW8.1 (Pin_1)
- new net: R35.1, U3.14 (Q5)
- new net: R35.2, ROW2.3 (Pin_3)
- new net: R47.1, U4.18 (Q1)
- new net: R47.2, ROW3.7 (Pin_7)
- new net: R51.1, U5.14 (Q5)
- new net: R51.2, ROW4.3 (Pin_3)
- new net: R63.1, U6.18 (Q1)
- new net: R63.2, ROW5.7 (Pin_7)
- new net: R82.1, U9.13 (Q6)
- new net: R83.1, U9.14 (Q5)
- new net: R84.1, U9.15 (Q4)
- new net: R85.1, U9.16 (Q3)
- new net: R86.1, U9.17 (Q2)
- new net: R87.1, U9.18 (Q1)
- new net: R88.1, U9.19 (Q0)
- new net: R32.2, ROW1.8 (Pin_8)
- new net: R80.1, U8.19 (Q0)
- new net: R80.2, ROW7.8 (Pin_8)
- new net: R59.1, U6.14 (Q5)
- new net: R59.2, ROW5.3 (Pin_3)
- new net: R57.2, ROW5.1 (Pin_1)
- new net: R58.2, ROW5.2 (Pin_2)
- new net: R60.2, ROW5.4 (Pin_4)
- new net: R61.2, ROW5.5 (Pin_5)
- new net: R62.2, ROW5.6 (Pin_6)
- new net: R64.2, ROW5.8 (Pin_8)
- new net: R54.1, U5.17 (Q2)
- new net: R54.2, ROW4.6 (Pin_6)
- new net: R33.2, ROW2.1 (Pin_1)
- new net: R34.2, ROW2.2 (Pin_2)
- new net: R36.2, ROW2.4 (Pin_4)
- new net: R37.2, ROW2.5 (Pin_5)
- new net: R38.2, ROW2.6 (Pin_6)
- new net: R39.2, ROW2.7 (Pin_7)
- new net: R40.2, ROW2.8 (Pin_8)
- new net: R87.2, ROW8.7 (Pin_7)
- new net: R44.1, U4.15 (Q4)
- new net: R44.2, ROW3.4 (Pin_4)
- new net: R61.1, U6.16 (Q3)
- new net: R67.1, U7.14 (Q5)
- new net: R67.2, ROW6.3 (Pin_3)
- new net: R76.1, U8.15 (Q4)
- new net: R76.2, ROW7.4 (Pin_4)
- new net: R73.2, ROW7.1 (Pin_1)
- new net: R74.2, ROW7.2 (Pin_2)
- new net: R75.2, ROW7.3 (Pin_3)
- new net: R77.2, ROW7.5 (Pin_5)
- new net: R78.2, ROW7.6 (Pin_6)
- new net: R79.2, ROW7.7 (Pin_7)
- new net: R39.1, U3.18 (Q1)
- new net: R83.2, ROW8.3 (Pin_3)
- new net: R88.2, ROW8.8 (Pin_8)
- new net: R53.1, U5.16 (Q3)
- new net: R53.2, ROW4.5 (Pin_5)
- new net: R41.1, U4.12 (Q7)
- new net: R42.1, U4.13 (Q6)
- new net: R43.1, U4.14 (Q5)
- new net: R45.1, U4.16 (Q3)
- new net: R46.1, U4.17 (Q2)
- new net: R48.1, U4.19 (Q0)
- new net: R85.2, ROW8.5 (Pin_5)
- new net: R82.2, ROW8.2 (Pin_2)
- new net: R84.2, ROW8.4 (Pin_4)
- new net: R86.2, ROW8.6 (Pin_6)
- new net: R66.2, ROW6.2 (Pin_2)
- new net: R68.2, ROW6.4 (Pin_4)
- new net: R69.2, ROW6.5 (Pin_5)
- new net: R72.2, ROW6.8 (Pin_8)
- new net: R34.1, U3.13 (Q6)
- new net: R38.1, U3.17 (Q2)
- new net: R62.1, U6.17 (Q2)
- new net: R40.1, U3.19 (Q0)
- new net: R73.1, U8.12 (Q7)
- new net: R55.1, U5.18 (Q1)
- new net: R55.2, ROW4.7 (Pin_7)
- new net: R79.1, U8.18 (Q1)
- new net: R43.2, ROW3.3 (Pin_3)
- new net: R27.2, ROW1.3 (Pin_3)
- new net: R46.2, ROW3.6 (Pin_6)
- new net: R60.1, U6.15 (Q4)
- new net: R78.1, U8.17 (Q2)
- new net: R74.1, U8.13 (Q6)
- new net: R72.1, U7.19 (Q0)
- new net: R25.2, ROW1.1 (Pin_1)
- new net: R69.1, U7.16 (Q3)
- new net: R26.2, ROW1.2 (Pin_2)
- new net: R52.1, U5.15 (Q4)
- new net: R52.2, ROW4.4 (Pin_4)
- new net: R66.1, U7.13 (Q6)
- new net: R68.1, U7.15 (Q4)
- new net: R36.1, U3.15 (Q4)
- new net: R58.1, U6.13 (Q6)
- new net: R37.1, U3.16 (Q3)
- new net: R33.1, U3.12 (Q7)
- new net: R29.2, ROW1.5 (Pin_5)
- new net: R64.1, U6.19 (Q0)
- new net: R41.2, ROW3.1 (Pin_1)
- new net: R31.2, ROW1.7 (Pin_7)
- new net: R77.1, U8.16 (Q3)
- new net: R42.2, ROW3.2 (Pin_2)
- new net: R49.1, U5.12 (Q7)
- new net: R49.2, ROW4.1 (Pin_1)
- new net: R48.2, ROW3.8 (Pin_8)
- new net: R57.1, U6.12 (Q7)
- new net: R45.2, ROW3.5 (Pin_5)
- new net: R50.1, U5.13 (Q6)
- new net: R56.1, U5.19 (Q0)
- new net: R50.2, ROW4.2 (Pin_2)
- new net: R56.2, ROW4.8 (Pin_8)
- new net: R75.1, U8.14 (Q5)
Other:
- moved on the sheet: A1, C1, C10, C11, C12, C2, C3, C4, C5, C6, C7, C8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

Commit message: update
Parts:
- C10: footprint Capacitor_THT:CP_Axial_L10.0mm_D4.5mm_P15.00mm_Horizontal -> Capacitor_THT:CP_Radial_D4.0mm_P1.50mm
- J1, ROW1, ROW2, ROW3, ROW4, ROW5, ROW6, ROW7, ROW8: footprint Connector_PinHeader_1.00mm:PinHeader_1x08_P1.00mm_Horizontal -> Connector_PinHeader_1.00mm:PinHeader_1x08_P1.00mm_Vertical
- R1, R10, R11, R12, R13, R14, R15, R16, R17, R18, R2, R3, R4, R5, R6, R7, R8, R9: footprint Resistor_SMD:R_0815_2038Metric_Pad1.20x4.05mm_HandSolder -> Resistor_SMD:R_0805_2012Metric_Pad1.20x1.40mm_HandSolder
- R19, R20, R21, R22, R23, R24, R25, R26, R27, R28, R29, R30, R31, R32, R33, R34, R35, R36, R37, R38, R39, R40, R41, R42, R43, R44, R45, R46, R47, R48, R49, R50, R51, R52, R53, R54, R55, R56, R57, R58, R59, R60, R61, R62, R63, R64, R65, R66, R67, R68, R69, R70, R71, R72, R73, R74, R75, R76, R77, R78, R79, R80, R81, R82, R83, R84, R85, R86, R87, R88: footprint Resistor_SMD:R_0815_2038Metric -> Resistor_SMD:R_0805_2012Metric_Pad1.20x1.40mm_HandSolder
- U9: footprint DIP254P762X420-20 -> 74HC574N:DIP254P762X420-20

Commit message: Update Matrix.kicad_sch
Parts:
- removed A1: Arduino_Nano_v3.x, Module:Arduino_Nano, symbol MCU_Module:Arduino_Nano_v3.x
- added U10: ESP32-S3, Package_DFN_QFN:QFN-56-1EP_7x7mm_P0.4mm_EP4x4mm, symbol MCU_Espressif:ESP32-S3
- C1, C2, C3, C4, C5, C6, C7, C8, C9: value C -> 0.1uf
Connections:
- net A1: now also U10.14 (GPIO9)
- net A2: now also U10.15 (GPIO10)
- net A3: now also U10.16 (GPIO11)
- net D0: now also U10.6 (GPIO1)
- net D1: now also U10.7 (GPIO2)
- net D2: now also U10.8 (GPIO3)
- net D3: now also U10.9 (GPIO4)
- net D4: now also U10.10 (GPIO5)
- net D5: now also U10.11 (GPIO6)
- net D6: now also U10.12 (GPIO7)
- net D7: now also U10.13 (GPIO8)
- net OE: now also U10.18 (GPIO13)
- new net: U10.2 (VDD3P3), U10.3 (VDD3P3)
- new net: U10.55 (VDDA), U10.56 (VDDA)
- new net CATHODE1: U10.19 (GPIO14)
- new net CATHODE2: U10.21 (XTAL_32K_P/GPIO15)
- new net CATHODE3: U10.22 (XTAL_32K_N/GPIO16)
- new net CATHODE4: U10.23 (GPIO17)
- new net CATHODE5: U10.24 (GPIO18)
- new net CATHODE6: U10.27 (GPIO21)
- new net CATHODE7: U10.37 (SPICLK_P/GPIO47)
- new net CATHODE8: U10.36 (SPICLK_N/GPIO48)
Other:
- moved on the sheet: J1, Q1, Q10, Q11, Q12, Q13, Q14, Q15, Q16, Q2, Q3, Q4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

Commit message: Update Matrix.kicad_sch
Connections:
- net GND: now also U1.8 (GND)
Other:
- moved on the sheet: C1, C10, C11, C12, C2, C3, C4, C5, C6, C7, C8, C9
