File: Matrix/.history/Matrix.kicad_sch (KiCad schematic)
At the start: 146 parts, among them J1 Conn_01x08, Q1 2N2219, Q10 2N2219, Q11 2N2219, Q12 2N2219, Q13 2N2219, Q14 2N2219, Q15 2N2219, Q16 2N2219, Q2 2N2219, Q3 2N2219, Q4 2N2219, Q5 2N2219, Q6 2N2219, Q7 2N2219, Q8 2N2219, Q9 2N2219, U1 74HC138, U10 ESP32-S3, U2 74HC574N, U3 74HC574N, U4 74HC574N, U5 74HC574N, U6 74HC574N, U7 74HC574N, U8 74HC574N, U9 74HC574N

Commit message: Update Matrix.kicad_sch
Parts:
- added C23: 22uf, symbol Device:C
- added D1: SS34, Diode_SMD:D_SMA, symbol Diode:SS34
- added J2: USB_C_Receptacle_USB2.0_16P, symbol Connector:USB_C_Receptacle_USB2.0_16P
- added R89, R90: 5.1k, symbol Device:R
- added U11: AP2112K-3.3, Package_TO_SOT_SMD:SOT-23-5, symbol Regulator_Linear:AP2112K-3.3
Connections:
- net +3.3V: now also U11.5 (VOUT)
- net +5V: now also C23.1, D1.1 (K), U11.1 (VIN)
- net GND: now also C23.2, J2.A1 (GND), J2.A12 (GND), J2.B1 (GND), J2.B12 (GND), J2.SH (SHIELD), R89.1, R90.1, U11.2 (GND)
- net D-: now reaches U10.25 (GPIO19/USB_D-)
- net D-: now also J2.A7 (D-), J2.B7 (D-)
- net D+: now reaches U10.26 (GPIO20/USB_D+)
- net D+: now also J2.A6 (D+), J2.B6 (D+)
- new net: J2.B5 (CC2), R90.2
- new net: J2.A5 (CC1), R89.2
- new net: D1.2 (A), J2.A4 (VBUS), J2.A9 (VBUS), J2.B4 (VBUS), J2.B9 (VBUS)
- no-connect marks 0 -> 2

Commit message: Update Matrix.kicad_sch
Parts:
- added AE1: Antenna_Chip, symbol Device:Antenna_Chip
- added C24, C25: 10uf, symbol Device:C
- added C26: 100nf, symbol Device:C
- added C27, C28: 12pf, symbol Device:C
- added C29, C30, C31, C32: 1.5pf, symbol Device:C
- added D2: ESD9B3.3ST5G, Diode_SMD:D_SOD-923, symbol Diode:ESD9B3.3ST5G
- added L2: 24 nh, symbol Device:L
- added L3: 2.7nh, symbol Device:L
- added L4: 2.2nh, symbol Device:L
- added U13: W25Q32JVSS, Package_SO:SOIC-8_5.3x5.3mm_P1.27mm, symbol Memory_Flash:W25Q32JVSS
- added Y1: 40MHz, symbol Device:Crystal
Connections:
- net +3.3V: now also C21.1, C22.1, U10.29 (VDD_SPI), C25.1, C26.1, U13.8 (VCC)
- net +5V: now also U11.3 (EN), C24.2
- net GND: now also AE1.1 (FEED), C24.1, C25.2, C26.2, C27.1, C28.1, C29.2, C30.2, C31.2, C32.2, D2.1 (A1), U13.4 (GND)
- net at U10.1 (LNA_IN): now also C29.1, L3.1
- net SPIHD: now reaches U10.30 (SPIHD)
- net SPIHD: now also U13.7 (~{HOLD}/~{RESET}/IO_{3})
- net SPICS0: now reaches U10.32 (SPICS0)
- net SPICS0: now also U13.1 (~{CS})
- net SPICLK: now reaches U10.33 (SPICLK)
- net SPICLK: now also U13.6 (CLK)
- net SPIQ: now reaches U10.34 (SPIQ)
- net SPIQ: now also U13.2 (DO/IO_{1})
- net SPID: now reaches U10.35 (SPID)
- net SPID: now also U13.5 (DI/IO_{0})
- net at U10.53 (XTAL_N): now also C28.2, Y1.1
- net at U10.54 (XTAL_P): now also L2.2
- new net: C27.2, L2.1, Y1.2
- new net: C30.1, C31.1, L3.2, L4.1
- new net: AE1.2 (PCB_Trace), C32.1, D2.2 (A2), L4.2
- new net SPIWP: U13.3 (~{WP}/IO_{2})
Other:
- note added: "FLASH"
- note added: "Power Supply"
- moved on the sheet: C23, D1, J2, R89, R90, U11

Commit message: Update Matrix.kicad_sch
Other:
- note added: "(Near VCC of 74HC574's and 74HC138) 0.1uf x 9"
- note added: "ESP-32 S3"
- moved on the sheet: AE1, C1, C10, C11, C12, C13, C14, C15, C16, C17, C18, C19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

Commit message: Update Matrix.kicad_sch
Parts:
- L1: value 2.0nH(0.1nH) 500mA -> 2.0nh(0.1nh) 500mA
- L2: value 24 nh -> 24nh
- Y1: value 40MHz -> 40MHz (+-10ppm)
Other:
- moved on the sheet: C23, C24, C25, C26, D1, J2, R89, R90, U11

Commit message: Update Matrix.kicad_sch
Parts:
- added C33: C, symbol Device:C
Connections:
- net +3.3V: now also U1.16 (VCC), U1.6 (E2), U2.20 (VCC), U3.20 (VCC), U4.20 (VCC), U5.20 (VCC), U6.20 (VCC), U7.20 (VCC), U8.20 (VCC), U9.20 (VCC)
- net +5V: no longer U1.4 (~{E0})
- net GND: now also U1.4 (~{E0}); no longer U1.6 (E2), U2.20 (VCC), U3.20 (VCC), U4.20 (VCC), U5.20 (VCC), U6.20 (VCC), U7.20 (VCC), U8.20 (VCC), U9.20 (VCC)

Commit message: Update Matrix.kicad_sch
Parts:
- removed C33: C, symbol Device:C
- added U12: ER_OLEDM0.91_1x-I2C, Display:ER_OLEDM0.91_1x-I2C, symbol Display_Graphic:ER_OLEDM0.91_1x-I2C
Connections:
- net CATHODE1 is gone; now on net CATHODE 1: U10.19 (GPIO14)
- net CATHODE2 is gone; now on net CATHODE 2: U10.21 (XTAL_32K_P/GPIO15)
- net CATHODE3 is gone; now on net CATHODE 3: U10.22 (XTAL_32K_N/GPIO16)
- net CATHODE4 is gone; now on net CATHODE 4: U10.23 (GPIO17)
- net CATHODE5 is gone; now on net CATHODE 5: U10.24 (GPIO18)
- net CATHODE6 is gone; now on net CATHODE 6: U10.27 (GPIO21)
- net CATHODE7 is gone; now on net CATHODE 7: U10.37 (SPICLK_P/GPIO47)
- net CATHODE8 is gone; now on net CATHODE 8: U10.36 (SPICLK_N/GPIO48)
- net +3.3V: now also U12.2 (VCC)
- net GND: now also AE1.2 (PCB_Trace), U12.1 (GND); no longer AE1.1 (FEED)
- net SPIWP: now also U10.31 (SPIWP)
- net SDA: now reaches U10.40 (GPIO35)
- net SDA: now also U12.4 (SDA)
- net SCL: now reaches U10.41 (GPIO36)
- net SCL: now also U12.3 (SCL)
- net at C32.1, D2.2 (A2), L4.2: now also AE1.1 (FEED); no longer AE1.2 (PCB_Trace)
- no-connect marks 2 -> 18
Other:
- note added: "OLED display"
- moved on the sheet: AE1, C13, C14, C15, C16, C17, C18, C19, C20, C21, C22, C24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

Commit message: Update Matrix.kicad_sch
Parts:
- AE1: footprint (none) -> AH316M245001-T:ANTC3216X60N
- C13, C14, C15, C16, C17, C18, C19, C20, C21, C22, C23, C24, C25, C26, C27, C28, C29, C30, C31, C32: footprint (none) -> Capacitor_SMD:C_0805_2012Metric_Pad1.18x1.45mm_HandSolder
- J2: footprint (none) -> Connector_USB:USB_C_Receptacle_GCT_USB4105-xx-A_16P_TopMnt_Horizontal
- L1, L2, L3, L4: footprint (none) -> Inductor_SMD:L_0805_2012Metric_Pad1.05x1.20mm_HandSolder
- R89, R90: footprint (none) -> Resistor_SMD:R_0805_2012Metric_Pad1.20x1.40mm_HandSolder
- Y1: footprint (none) -> Crystal:Crystal_SMD_3225-4Pin_3.2x2.5mm_HandSoldering
Changed lines of the file:
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@@
 			)
 		)
-		(property "Footprint" ""
+		(property "Footprint" "Resistor_SMD:R_0805_2012Metric_Pad1.20x1.40mm_HandSolder"
 			(at 387.35 64.262 90)
 			(hide yes)
@@
 			)
 		)
-		(property "Footprint" ""
+		(property "Footprint" "Capacitor_SMD:C_0805_2012Metric_Pad1.18x1.45mm_HandSolder"
 			(at 157.1752 551.18 0)
 			(hide yes)
@@
 			)
 		)
-		(property "Footprint" ""
+		(property "Footprint" "Crystal:Crystal_SMD_3225-4Pin_3.2x2.5mm_HandSoldering"
 			(at 62.23 547.37 0)
 			(hide yes)
@@
 			)
 		)
-		(property "Footprint" ""
+		(property "Footprint" "Inductor_SMD:L_0805_2012Metric_Pad1.05x1.20mm_HandSolder"
 			(at 104.14 440.69 0)
 			(hide yes)
@@
 			)
 		)
-		(property "Footprint" ""
+		(property "Footprint" "Capacitor_SMD:C_0805_2012Metric_Pad1.18x1.45mm_HandSolder"
 			(at 68.2752 448.31 0)
 			(hide yes)
@@
 			)
 		)
-		(property "Footprint" ""
+		(property "Footprint" "Capacitor_SMD:C_0805_2012Metric_Pad1.18x1.45mm_HandSolder"
 			(at 403.5552 52.07 0)
 			(hide yes)
@@
 			)
 		)
-		(property "Footprint" ""
+		(property "Footprint" "Capacitor_SMD:C_0805_2012Metric_Pad1.18x1.45mm_HandSolder"
 			(at 55.88 552.7548 0)
 			(hide yes)
@@
 			)
 		)
-		(property "Footprint" ""
+		(property "Footprint" "Capacitor_SMD:C_0805_2012Metric_Pad1.18x1.45mm_HandSolder"
 			(at 143.2052 438.15 0)
 			(hide yes)
@@
 			)
 		)
-		(property "Footprint" ""
+		(property "Footprint" "Resistor_SMD:R_0805_2012Metric_Pad1.20x1.40mm_HandSolder"
 			(at 387.35 61.722 90)
 			(hide yes)
@@
 			)
 		)
-		(property "Footprint" ""
+		(property "Footprint" "Capacitor_SMD:C_0805_2012Metric_Pad1.18x1.45mm_HandSolder"
 			(at 91.1352 471.17 0)
 			(hide yes)
@@
 			)
 		)
-		(property "Footprint" ""
+		(property "Footprint" "Capacitor_SMD:C_0805_2012Metric_Pad1.18x1.45mm_HandSolder"
 			(at 93.6752 448.31 0)
 			(hide yes)
@@
 			)
 		)
-		(property "Footprint" ""
+		(property "Footprint" "Inductor_SMD:L_0805_2012Metric_Pad1.05x1.20mm_HandSolder"
 			(at 72.39 541.02 0)
 			(hide yes)
@@
 			)
 		)
-		(property "Footprint" ""
+		(property "Footprint" "Capacitor_SMD:C_0805_2012Metric_Pad1.18x1.45mm_HandSolder"
 			(at 177.4952 551.18 0)
 			(hide yes)
@@
 			)
 		)
-		(property "Footprint" ""
+		(property "Footprint" "Capacitor_SMD:C_0805_2012Metric_Pad1.18x1.45mm_HandSolder"
 			(at 444.1952 106.68 0)
 			(hide yes)
@@
 			)
 		)
-		(property "Footprint" ""
+		(property "Footprint" "Capacitor_SMD:C_0805_2012Metric_Pad1.18x1.45mm_HandSolder"
 			(at 115.2652 448.31 0)
 			(hide yes)
@@
 			)
 		)
-		(property "Footprint" ""
+		(property "Footprint" "Capacitor_SMD:C_0805_2012Metric_Pad1.18x1.45mm_HandSolder"
 			(at 205.4352 551.18 0)
 			(hide yes)
@@
 			)
 		)
-		(property "Footprint" ""
+		(property "Footprint" "Capacitor_SMD:C_0805_2012Metric_Pad1.18x1.45mm_HandSolder"
 			(at 435.3052 106.68 0)
 			(hide yes)
@@
 			)
 		)
-		(property "Footprint" ""
+		(property "Footprint" "Capacitor_SMD:C_0805_2012Metric_Pad1.18x1.45mm_HandSolder"
 			(at 402.2852 99.06 0)
 			(hide yes)
@@
 			)
 		)
-		(property "Footprint" ""
+		(property "Footprint" "Inductor_SMD:L_0805_2012Metric_Pad1.05x1.20mm_HandSolder"
 			(at 195.58 543.56 0)
 			(hide yes)
@@
 			)
 		)
-		(property "Footprint" ""
+		(property "Footprint" "Capacitor_SMD:C_0805_2012Metric_Pad1.18x1.45mm_HandSolder"
 			(at 140.6652 464.82 0)
 			(hide yes)
@@
 			)
 		)
-		(property "Footprint" ""
+		(property "Footprint" "Inductor_SMD:L_0805_2012Metric_Pad1.05x1.20mm_HandSolder"
 			(at 167.64 543.56 0)
 			(hide yes)
@@
 			)
 		)
-		(property "Footprint" ""
+		(property "Footprint" "Capacitor_SMD:C_0805_2012Metric_Pad1.18x1.45mm_HandSolder"
 			(at 136.8552 438.15 0)
 			(hide yes)
@@
 			)
 		)
-		(property "Footprint" ""
+		(property "Footprint" "Capacitor_SMD:C_0805_2012Metric_Pad1.18x1.45mm_HandSolder"
 			(at 55.88 540.0548 0)
 			(hide yes)
@@
 			)
 		)
-		(property "Footprint" ""
+		(property "Footprint" "Capacitor_SMD:C_0805_2012Metric_Pad1.18x1.45mm_HandSolder"
 			(at 103.8352 471.17 0)
 			(hide yes)
@@
 			)
 		)
-		(property "Footprint" ""
+		(property "Footprint" "Connector_USB:USB_C_Receptacle_GCT_USB4105-xx-A_16P_TopMnt_Horizontal"
 			(at 369.57 73.66 0)
 			(hide yes)
@@
 			)
 		)
-		(property "Footprint" ""
+		(property "Footprint" "Capacitor_SMD:C_0805_2012Metric_Pad1.18x1.45mm_HandSolder"
 			(at 186.3852 551.18 0)
 			(hide yes)
@@
 			)
 		)
-		(property "Footprint" ""
+		(property "Footprint" "Capacitor_SMD:C_0805_2012Metric_Pad1.18x1.45mm_HandSolder"
 			(at 150.8252 464.82 0)
 			(hide yes)
@@
 			)
 		)
-		(property "Footprint" ""
+		(property "Footprint" "Capacitor_SMD:C_0805_2012Metric_Pad1.18x1.45mm_HandSolder"
 			(at 80.9752 448.31 0)
 			(hide yes)
@@
 			)
 		)
-		(property "Footprint" ""
+		(property "Footprint" "AH316M245001-T:ANTC3216X60N"
 			(at 236.22 536.575 0)
 			(hide yes)
