File: Matrix/.history/Matrix.kicad_pcb (KiCad board)
At the start: 2 copper layers, 169 parts, among them J1 Conn_01x08, J2 USB_C_Receptacle_USB2.0_16P, Q1 2N2219, Q10 2N2219, Q11 2N2219, Q12 2N2219, Q13 2N2219, Q14 2N2219, Q15 2N2219, Q16 2N2219, Q2 2N2219, Q3 2N2219, Q4 2N2219, Q5 2N2219, Q6 2N2219, Q7 2N2219, Q8 2N2219, Q9 2N2219, U1 74HC138, U10 ESP32-S3, U11 AP2112K-3.3, U12 ER_OLEDM0.91_1x-I2C, U13 W25Q32JVSS, U2 74HC574N, U3 74HC574N, U4 74HC574N, U5 74HC574N, U6 74HC574N, U7 74HC574N, U8 74HC574N, U9 74HC574N, Y1 40MHz (+-10ppm)

Commit message: Update Matrix.kicad_pcb
Parts:
- moved C15 20.5 mm to (102.0, 316.2)
- moved C16 20.5 mm to (102.0, 319.2)
- moved C17 8.65 mm to (103.8, 331.4)
- moved C18 8.65 mm to (103.8, 334.4)
- moved L1 1.33 mm to (87.8, 330.5)
- moved C29 0.39 mm to (103.9, 311.7), turned to 180 degrees
- moved C31 0.14 mm to (103.8, 308.5)
Changed lines of the file:
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@@
 	(footprint "Capacitor_SMD:C_0805_2012Metric_Pad1.18x1.45mm_HandSolder"
 		(layer "F.Cu")
-		(at 109.2075 327.58)
+		(at 103.8325 334.36)
 		(descr "Capacitor SMD 0805 (2012 Metric), square (rectangular) end terminal, IPC-7351 nominal with elongated pad for handsoldering. (Body size source: IPC-SM-782 page 76, https://www.pcb-3d.com/wordpress/wp-content/uploads/ipc-sm-782a_amendment_1_and_2.pdf, https://docs.google.com/spreadsheets/d/1BsfQQcO9C6DZCsRaXUlFlo91Tg2WpOkGARC1WS5S8t0/edit?usp=sharing)")
 		(tags "capacitor handsolder")
@@
 	(footprint "Capacitor_SMD:C_0805_2012Metric_Pad1.18x1.45mm_HandSolder"
 		(layer "F.Cu")
-		(at 109.2075 324.57)
+		(at 103.8325 331.35)
 		(descr "Capacitor SMD 0805 (2012 Metric), square (rectangular) end terminal, IPC-7351 nominal with elongated pad for handsoldering. (Body size source: IPC-SM-782 page 76, https://www.pcb-3d.com/wordpress/wp-content/uploads/ipc-sm-782a_amendment_1_and_2.pdf, https://docs.google.com/spreadsheets/d/1BsfQQcO9C6DZCsRaXUlFlo91Tg2WpOkGARC1WS5S8t0/edit?usp=sharing)")
 		(tags "capacitor handsolder")
@@
 	(footprint "Inductor_SMD:L_0805_2012Metric_Pad1.05x1.20mm_HandSolder"
 		(layer "F.Cu")
-		(at 88.4025 329.28)
+		(at 87.8275 330.48)
 		(descr "Inductor SMD 0805 (2012 Metric), square (rectangular) end terminal, IPC-7351 nominal with elongated pad for handsoldering. (Body size source: IPC-SM-782 page 80, https://www.pcb-3d.com/wordpress/wp-content/uploads/ipc-sm-782a_amendment_1_and_2.pdf)")
 		(tags "inductor handsolder")
@@
 	(footprint "Capacitor_SMD:C_0805_2012Metric_Pad1.18x1.45mm_HandSolder"
 		(layer "F.Cu")
-		(at 104.3975 336.61)
+		(at 102.0025 316.22)
 		(descr "Capacitor SMD 0805 (2012 Metric), square (rectangular) end terminal, IPC-7351 nominal with elongated pad for handsoldering. (Body size source: IPC-SM-782 page 76, https://www.pcb-3d.com/wordpress/wp-content/uploads/ipc-sm-782a_amendment_1_and_2.pdf, https://docs.google.com/spreadsheets/d/1BsfQQcO9C6DZCsRaXUlFlo91Tg2WpOkGARC1WS5S8t0/edit?usp=sharing)")
 		(tags "capacitor handsolder")
@@
 	(footprint "Capacitor_SMD:C_0805_2012Metric_Pad1.18x1.45mm_HandSolder"
 		(layer "F.Cu")
-		(at 103.8425 312.07)
+		(at 103.8925 311.68 180)
 		(descr "Capacitor SMD 0805 (2012 Metric), square (rectangular) end terminal, IPC-7351 nominal with elongated pad for handsoldering. (Body size source: IPC-SM-782 page 76, https://www.pcb-3d.com/wordpress/wp-content/uploads/ipc-sm-782a_amendment_1_and_2.pdf, https://docs.google.com/spreadsheets/d/1BsfQQcO9C6DZCsRaXUlFlo91Tg2WpOkGARC1WS5S8t0/edit?usp=sharing)")
 		(tags "capacitor handsolder")
@@
 		(duplicate_pad_numbers_are_jumpers no)
 		(fp_line
-			(start -0.261252 -0.735)
-			(end 0.261252 -0.735)
+			(start -0.261252 0.735)
+			(end 0.261252 0.735)
 			(stroke
 				(width 0.12)
@@
 		)
 		(fp_line
-			(start -0.261252 0.735)
-			(end 0.261252 0.735)
+			(start -0.261252 -0.735)
+			(end 0.261252 -0.735)
 			(stroke
 				(width 0.12)
@@
 		)
 		(pad "1" smd roundrect
-			(at -1.0375 0)
+			(at -1.0375 0 180)
 			(size 1.175 1.45)
 			(layers "F.Cu" "F.Mask" "F.Paste")
@@
 		)
 		(pad "2" smd roundrect
-			(at 1.0375 0)
+			(at 1.0375 0 180)
 			(size 1.175 1.45)
 			(layers "F.Cu" "F.Mask" "F.Paste")
@@
 	(footprint "Capacitor_SMD:C_0805_2012Metric_Pad1.18x1.45mm_HandSolder"
 		(layer "F.Cu")
-		(at 103.68 308.58)
+		(at 103.7825 308.49)
 		(descr "Capacitor SMD 0805 (2012 Metric), square (rectangular) end terminal, IPC-7351 nominal with elongated pad for handsoldering. (Body size source: IPC-SM-782 page 76, https://www.pcb-3d.com/wordpress/wp-content/uploads/ipc-sm-782a_amendment_1_and_2.pdf, https://docs.google.com/spreadsheets/d/1BsfQQcO9C6DZCsRaXUlFlo91Tg2WpOkGARC1WS5S8t0/edit?usp=sharing)")
 		(tags "capacitor handsolder")
@@
 	(footprint "Capacitor_SMD:C_0805_2012Metric_Pad1.18x1.45mm_HandSolder"
 		(layer "F.Cu")
-		(at 104.3975 339.62)
+		(at 102.0025 319.23)
 		(descr "Capacitor SMD 0805 (2012 Metric), square (rectangular) end terminal, IPC-7351 nominal with elongated pad for handsoldering. (Body size source: IPC-SM-782 page 76, https://www.pcb-3d.com/wordpress/wp-content/uploads/ipc-sm-782a_amendment_1_and_2.pdf, https://docs.google.com/spreadsheets/d/1BsfQQcO9C6DZCsRaXUlFlo91Tg2WpOkGARC1WS5S8t0/edit?usp=sharing)")
 		(tags "capacitor handsolder")

Commit message: Update Matrix.kicad_pcb
Parts:
- moved C20 280.5 mm to (294.2, 229.3), turned to 90 degrees
- moved C19 276.4 mm to (291.2, 229.3), turned to 90 degrees
- moved ROW4 264.4 mm to (237.8, 196.0)
- moved ROW3 244.0 mm to (221.3, 196.2)
- moved R49 240.4 mm to (242.4, 176.5)
- moved R50 240.4 mm to (242.4, 173.5)
- moved R51 240.4 mm to (242.4, 170.6)
- moved R52 240.4 mm to (242.4, 167.6)
- moved R53 240.4 mm to (242.4, 164.3)
- moved R54 240.4 mm to (242.4, 161.4)
- moved R55 240.4 mm to (242.4, 158.4)
- moved R56 240.4 mm to (242.4, 155.5)
- moved U5 235.3 mm to (238.3, 177.5)
- moved U12 233.7 mm to (266.9, 246.3)
- moved L1 222.7 mm to (286.8, 230.5), turned to 180 degrees
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Connections:
- C1 pad 1: +5V -> +3.3V
- C2 pad 1: +5V -> +3.3V
- C3 pad 1: +5V -> +3.3V
- C4 pad 1: +5V -> +3.3V
- C5 pad 1: +5V -> +3.3V
- C6 pad 1: +5V -> +3.3V
- C7 pad 1: +5V -> +3.3V
- C8 pad 1: +5V -> +3.3V
- C9 pad 1: +5V -> +3.3V
Other:
- board outline added: 150 x 150 mm

Commit message: Update Matrix.kicad_pcb
Parts:
- added C33: 10uf, Capacitor_SMD:C_0805_2012Metric_Pad1.18x1.45mm_HandSolder, F.Cu at (223.5, 235.1)
- added R91: 10k, Resistor_SMD:R_0805_2012Metric_Pad1.20x1.40mm_HandSolder, F.Cu at (223.6, 230.5)
- added SW1: SW_Push, Button_Switch_SMD:SW_SPST_PTS645Sx43SMTR92, B.Cu at (202.4, 232.5)
- added SW2: SW_Push, Button_Switch_SMD:SW_SPST_PTS645Sx43SMTR92, B.Cu at (216.2, 232.7)
- moved U13 78.8 mm to (206.6, 206.5)
- moved L2 76.7 mm to (193.7, 218.6)
- moved C22 76.7 mm to (215.7, 217.2)
- moved D2 76.7 mm to (195.0, 239.1)
- moved C14 76.7 mm to (199.2, 227.1)
- moved C18 76.7 mm to (212.6, 240.1)
- moved C28 76.7 mm to (193.8, 226.3)
- moved C29 76.7 mm to (205.0, 234.2)
- moved L3 76.7 mm to (205.6, 238.8)
- moved AE1 76.7 mm to (202.7, 243.8)
- moved C13 76.7 mm to (199.2, 230.1)
- moved C16 76.7 mm to (212.6, 236.1)
- moved C27 76.7 mm to (193.8, 223.3)
- moved C31 76.7 mm to (201.8, 234.3)
- moved L1 76.7 mm to (211.3, 243.9)
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Connections:
- U10 pad 4: unconnected-(U10-CHIP_PU-Pad4) -> Net-(U10-CHIP_PU)
- U10 pad 5: unconnected-(U10-GPIO0-Pad5) -> Net-(U10-GPIO0)
Routing:
- net D0: track 0.00 -> 236.3 mm, vias 0 -> 2
- net OE: track 0.00 -> 228.4 mm, vias 0 -> 7
- net D1: track 0.00 -> 227.0 mm, vias 0 -> 2
- net D2: track 0.00 -> 222.7 mm, vias 0 -> 4
- net D3: track 0.00 -> 220.0 mm, vias 0 -> 4
- net D4: track 0.00 -> 217.2 mm, vias 0 -> 4
- net D5: track 0.00 -> 211.1 mm, vias 0 -> 2
- net D6: track 0.00 -> 207.6 mm, vias 0 -> 2
- net D7: track 0.00 -> 204.5 mm, vias 0 -> 5
- net +5V: track 0.00 -> 200.2 mm, vias 0 -> 6
- net CATHODE 8: track 0.00 -> 163.9 mm, vias 0 -> 2
- net CATHODE 7: track 0.00 -> 152.8 mm, vias 0 -> 4
- net CATHODE 1: track 0.00 -> 139.2 mm
- net CATHODE 6: track 0.00 -> 135.2 mm, vias 0 -> 2
- net CATHODE 2: track 0.00 -> 127.3 mm, vias 0 -> 2
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- added copper zone on F.Cu, net +3.3V
- added copper zone on B.Cu, net GND
