File: Matrix/Matrix.kicad_sch (KiCad schematic)
At the start: 0 parts

Commit message: Update Matrix.kicad_sch
Parts:
- added U1: ESP32-S3, Package_DFN_QFN:QFN-56-1EP_7x7mm_P0.4mm_EP4x4mm, symbol MCU_Espressif:ESP32-S3
Connections:
- new net: U1.2 (VDD3P3), U1.3 (VDD3P3)
- new net: U1.55 (VDDA), U1.56 (VDDA)
Changed lines of the file:
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@@
 	(generator "eeschema")
 	(generator_version "10.0")
-	(paper "A4")
+	(paper "A2")
+	(symbol
+		(lib_id "MCU_Espressif:ESP32-S3")
+		(at 283.21 76.2 0)
+		(unit 1)
+		(body_style 1)
+		(exclude_from_sim no)
+		(in_bom yes)
+		(on_board yes)
+		(in_pos_files yes)
+		(dnp no)
+		(fields_autoplaced yes)
+		(property "Reference" "U1"
+			(at 285.3533 114.3 0)
+			(show_name no)
+			(do_not_autoplace no)
+			(effects
+				(font
+					(size 1.27 1.27)
+				)
+				(justify left)
+			)
+		)
+		(property "Value" "ESP32-S3"
+			(at 285.3533 116.84 0)
+			(show_name no)
+			(do_not_autoplace no)
+			(effects
+				(font
+					(size 1.27 1.27)
+				)
+				(justify left)
+			)
+		)
+		(property "Footprint" "Package_DFN_QFN:QFN-56-1EP_7x7mm_P0.4mm_EP4x4mm"
+			(at 284.48 128.016 0)
+			(hide yes)
+			(show_name no)
+			(do_not_autoplace no)
+			(effects
+				(font
+					(size 1.27 1.27)
+				)
+			)
+		)
+		(property "Datasheet" "https://www.espressif.com/sites/default/files/documentation/esp32-s3_datasheet_en.pdf"
+			(at 285.242 29.972 0)
+			(hide yes)
+			(show_name no)
+			(do_not_autoplace no)
+			(effects
+				(font
+					(size 1.27 1.27)
+				)
+			)
+		)
+		(property "Description" "Microcontroller, Wi-Fi 802.11b/g/n, Bluetooth, 32bit"
+			(at 282.448 32.512 0)
+			(hide yes)
+			(show_name no)
+			(do_not_autoplace no)
+			(effects
+				(font
+					(size 1.27 1.27)
+				)
+			)
+		)
+		(pin "3"
+		)
+		(pin "8"
+		)
+		(pin "10"
+		)
+		(pin "12"
+		)
+		(pin "15"
+		)
+		(pin "18"
+		)
+		(pin "22"
+		)
+		(pin "24"
+		)
+		(pin "9"
+		)
+		(pin "27"
+		)
+		(pin "30"
+		)
+		(pin "56"
+		)
+		(pin "34"
+		)
+		(pin "13"
+		)
+		(pin "36"
+		)
+		(pin "1"
+		)
+		(pin "5"
+		)
+		(pin "29"
+		)
+		(pin "31"
+		)
+		(pin "45"
+		)
+		(pin "2"
+		)
+		(pin "4"
+		)
+		(pin "7"
+		)
+		(pin "11"
+		)
+		(pin "6"
+		)
+		(pin "14"
+		)
+		(pin "16"
+		)
+		(pin "19"
+		)
+		(pin "20"
+		)
+		(pin "17"
+		)
+		(pin "51"
+		)
+		(pin "21"
+		)
+		(pin "23"
+		)
+		(pin "25"
+		)
+		(pin "26"
+		)
+		(pin "28"
+		)
+		(pin "32"
+		)
+		(pin "33"
+		)
+		(pin "35"
+		)
+		(pin "54"
+		)
+		(pin "53"
+		)
+		(pin "38"
+		)
+		(pin "44"
+		)
+		(pin "49"
+		)
+		(pin "50"
+		)
+		(pin "52"
+		)
+		(pin "47"
+		)
+		(pin "43"
+		)
+		(pin "55"
+		)
+		(pin "41"
+		)
+		(pin "39"
+		)
+		(pin "42"
+		)
+		(pin "37"
+		)
+		(pin "46"
+		)
+		(pin "48"
+		)
+		(pin "57"
+		)
+		(pin "40"
+		)
+		(instances
+			(project "Matrix"
+				(path "/88b088a6-0f2a-4bb0-891c-efec1204d77b"
+					(reference "U1")
+					(unit 1)
+				)
+			)
+		)
+	)
 	(sheet_instances
 		(path "/"

Commit message: Update Matrix.kicad_sch
Parts:
- removed U1: ESP32-S3, Package_DFN_QFN:QFN-56-1EP_7x7mm_P0.4mm_EP4x4mm, symbol MCU_Espressif:ESP32-S3
- added A1: Arduino_Nano_v3.x, Module:Arduino_Nano, symbol MCU_Module:Arduino_Nano_v3.x
- added C1, C2, C3, C4, C5, C6, C7, C8, C9: C, symbol Device:C
- added C10: 1000uf, symbol Device:C_Polarized_US
- added C11: 100uf, symbol Device:C_Polarized_US
- added C12: 10uf, symbol Device:C_Polarized_US
- added Q1, Q10, Q11, Q12, Q13, Q14, Q15, Q16, Q2, Q3, Q4, Q5, Q6, Q7, Q8, Q9: 2N2219, Package_TO_SOT_THT:TO-39-3, symbol Transistor_BJT:2N2219
Connections:
- new net: Q1.2 (B), Q2.2 (B), Q3.2 (B), Q4.2 (B), Q5.2 (B), Q6.2 (B), Q7.2 (B)
- new net +5V: C1.1, C10.1, C11.1, C12.1, C2.1, C3.1, C4.1, C5.1, C6.1, C7.1, C8.1, C9.1
- new net A1: A1.11 (D8)
- new net A2: A1.12 (D9)
- new net A3: A1.13 (D10)
- new net CATHODE 1: A1.19 (A0)
- new net CATHODE 2: A1.20 (A1)
- new net CATHODE 3: A1.21 (A2)
- new net CATHODE 4: A1.22 (A3)
- new net CATHODE 5: A1.23 (A4)
- new net CATHODE 6: A1.24 (A5)
- new net CATHODE 7: A1.15 (D12)
- new net CATHODE 8: A1.16 (D13)
- new net D0: A1.2 (D0/RX)
- new net D1: A1.1 (D1/TX)
- new net D2: A1.5 (D2)
- new net D3: A1.6 (D3)
- new net D4: A1.7 (D4)
- new net D5: A1.8 (D5)
- new net D6: A1.9 (D6)
- new net D7: A1.10 (D7)
- new net GND: C1.2, C10.2, C11.2, C12.2, C2.2, C3.2, C4.2, C5.2, C6.2, C7.2, C8.2, C9.2, Q1.1 (E), Q10.1 (E), Q11.1 (E), Q12.1 (E), Q13.1 (E), Q14.1 (E), Q15.1 (E), Q16.1 (E), Q4.1 (E), Q5.1 (E), Q6.1 (E), Q7.1 (E), Q8.1 (E), Q9.1 (E)
- new net OE: A1.14 (D11)

Commit message: Update Matrix.kicad_sch
Parts:
- added J1, ROW1, ROW2, ROW3, ROW4, ROW5, ROW6, ROW7, ROW8: Conn_01x08, Connector_PinHeader_1.00mm:PinHeader_1x08_P1.00mm_Vertical, symbol Connector_Generic:Conn_01x08
- added R1, R10, R11, R12, R13, R14, R15, R16, R2, R3, R4, R5, R6, R7, R8, R9: 1k, Resistor_SMD:R_0805_2012Metric_Pad1.20x1.40mm_HandSolder, symbol Device:R
- added R17, R18, R19, R20, R21, R22, R23, R24: 10k, Resistor_SMD:R_0805_2012Metric_Pad1.20x1.40mm_HandSolder, symbol Device:R
- added R25, R26, R27, R28, R29, R30, R31, R32, R33, R34, R35, R36, R37, R38, R39, R40, R41, R42, R43, R44, R45, R46, R47, R48, R49, R50, R51, R52, R53, R54, R55, R56, R57, R58, R59, R60, R61, R62, R63, R64, R65, R66, R67, R68, R69, R70, R71, R72, R73, R74, R75, R76, R77, R78, R79, R80, R81, R82, R83, R84, R85, R86, R87, R88: 100R, Resistor_SMD:R_0805_2012Metric_Pad1.20x1.40mm_HandSolder, symbol Device:R
- added U1: 74HC138, 74HC138D:SOIC127P600X175-16N, symbol 74xx:74HC138
- added U2, U3, U4, U5, U6, U7, U8, U9: 74HC574N, 74HC574N:DIP254P762X420-20, symbol 74HC574N:74HC574N
- C1, C2, C3, C4, C5, C6, C7, C8, C9: footprint (none) -> Capacitor_SMD:C_0805_2012Metric
- C10: footprint (none) -> Capacitor_THT:CP_Radial_D4.0mm_P1.50mm
- C11, C12: footprint (none) -> Capacitor_SMD:C_0805_2012Metric_Pad1.18x1.45mm_HandSolder
Connections:
- net +5V: now also R17.1, R18.1, R19.1, R20.1, R21.1, R22.1, R23.1, R24.1, U1.4 (~{E0})
- net A1: now also U1.1 (A0)
- net A2: now also U1.2 (A1)
- net A3: now also U1.3 (A2)
- net CATHODE 1: now also R1.1, R2.1
- net CATHODE 2: now also R3.1, R4.1
- net CATHODE 3: now also R5.1, R6.1
- net CATHODE 4: now also R7.1, R8.1
- net CATHODE 5: now also R10.1, R9.1
- net CATHODE 6: now also R11.1, R12.1
- net CATHODE 7: now also R13.1, R14.1
- net CATHODE 8: now also R15.1, R16.1
- net D0: now also U2.2 (D0), U3.2 (D0), U4.2 (D0), U5.2 (D0), U6.2 (D0), U7.2 (D0), U8.2 (D0), U9.2 (D0)
- net D1: now also U2.3 (D1), U3.3 (D1), U4.3 (D1), U5.3 (D1), U6.3 (D1), U7.3 (D1), U8.3 (D1), U9.3 (D1)
- net D2: now also U2.4 (D2), U3.4 (D2), U4.4 (D2), U5.4 (D2), U6.4 (D2), U7.4 (D2), U8.4 (D2), U9.4 (D2)
- net D3: now also U2.5 (D3), U3.5 (D3), U4.5 (D3), U5.5 (D3), U6.5 (D3), U7.5 (D3), U8.5 (D3), U9.5 (D3)
- net D4: now also U2.6 (D4), U3.6 (D4), U4.6 (D4), U5.6 (D4), U6.6 (D4), U7.6 (D4), U8.6 (D4), U9.6 (D4)
- net D5: now also U2.7 (D5), U3.7 (D5), U4.7 (D5), U5.7 (D5), U6.7 (D5), U7.7 (D5), U8.7 (D5), U9.7 (D5)
- net D6: now also U2.8 (D6), U3.8 (D6), U4.8 (D6), U5.8 (D6), U6.8 (D6), U7.8 (D6), U8.8 (D6), U9.8 (D6)
- net D7: now also U2.9 (D7), U3.9 (D7), U4.9 (D7), U5.9 (D7), U6.9 (D7), U7.9 (D7), U8.9 (D7), U9.9 (D7)
- net GND: now also Q2.1 (E), Q3.1 (E), U1.5 (~{E1}), U1.6 (E2), U2.10 (GND), U2.20 (VCC), U3.10 (GND), U3.20 (VCC), U4.10 (GND), U4.20 (VCC), U5.10 (GND), U5.20 (VCC), U6.10 (GND), U6.20 (VCC), U7.10 (GND), U7.20 (VCC), U8.10 (GND), U8.20 (VCC), U9.10 (GND), U9.20 (VCC)
- net OE: now also U2.1 (~{OE}), U3.1 (~{OE}), U4.1 (~{OE}), U5.1 (~{OE}), U6.1 (~{OE}), U7.1 (~{OE}), U8.1 (~{OE}), U9.1 (~{OE})
- net at Q1.3 (C): now also Q2.3 (C), J1.1 (Pin_1), R17.2
- net at Q13.2 (B): now also R13.2
- net at Q13.3 (C): now also Q14.3 (C), J1.7 (Pin_7), R23.2
- net at Q16.2 (B): now also R16.2
- net at Q16.3 (C): now also Q15.3 (C), J1.8 (Pin_8), R24.2
- net at Q11.2 (B): now also R11.2
- net at Q11.3 (C): now also Q12.3 (C), J1.6 (Pin_6), R22.2
- net at Q15.2 (B): now also R15.2
- net at Q7.3 (C): now also Q8.3 (C), J1.4 (Pin_4), R20.2
- net at Q5.3 (C): now also Q6.3 (C), J1.3 (Pin_3), R19.2
- net at Q8.2 (B): now also R8.2
- net at Q12.2 (B): now also R12.2
- net at Q14.2 (B): now also R14.2
- net at Q9.2 (B): now also R9.2
- net at Q9.3 (C): now also Q10.3 (C), J1.5 (Pin_5), R21.2
- net at Q10.2 (B): now also R10.2
- net at Q3.3 (C): now also Q4.3 (C), J1.2 (Pin_2), R18.2
- new net: R65.1, U7.12 (Q7)
- new net: R65.2, ROW6.1 (Pin_1)
- new net: R71.1, U7.18 (Q1)
- new net: R71.2, ROW6.7 (Pin_7)
- new net: Q5.2 (B), R5.2
- new net: R28.1, U2.15 (Q4)
- new net: R28.2, ROW1.4 (Pin_4)
- new net: R30.1, U2.17 (Q2)
- new net: R30.2, ROW1.6 (Pin_6)
- new net: R70.1, U7.17 (Q2)
- new net: R70.2, ROW6.6 (Pin_6)
- new net: U1.15 (~{Y0}), U2.11 (CP)
- new net: R25.1, U2.12 (Q7)
- new net: R26.1, U2.13 (Q6)
- new net: R27.1, U2.14 (Q5)
- new net: R29.1, U2.16 (Q3)
- new net: R31.1, U2.18 (Q1)
- new net: R32.1, U2.19 (Q0)
- new net: R81.1, U9.12 (Q7)
- new net: R81.2, ROW8.1 (Pin_1)
- new net: R35.1, U3.14 (Q5)
- new net: R35.2, ROW2.3 (Pin_3)
- new net: R47.1, U4.18 (Q1)
- new net: R47.2, ROW3.7 (Pin_7)
- new net: R51.1, U5.14 (Q5)
- new net: R51.2, ROW4.3 (Pin_3)
- new net: R63.1, U6.18 (Q1)
- new net: R63.2, ROW5.7 (Pin_7)
- new net: U1.7 (~{Y7}), U9.11 (CP)
- new net: R82.1, U9.13 (Q6)
- new net: R83.1, U9.14 (Q5)
- new net: R84.1, U9.15 (Q4)
- new net: R85.1, U9.16 (Q3)
- new net: R86.1, U9.17 (Q2)
- new net: R87.1, U9.18 (Q1)
- new net: R88.1, U9.19 (Q0)
- new net: R32.2, ROW1.8 (Pin_8)
- new net: R80.1, U8.19 (Q0)
- new net: R80.2, ROW7.8 (Pin_8)
- new net: R59.1, U6.14 (Q5)
- new net: R59.2, ROW5.3 (Pin_3)
- new net: Q1.2 (B), R1.2
- new net: R57.2, ROW5.1 (Pin_1)
- new net: R58.2, ROW5.2 (Pin_2)
- new net: R60.2, ROW5.4 (Pin_4)
- new net: R61.2, ROW5.5 (Pin_5)
- new net: R62.2, ROW5.6 (Pin_6)
- new net: R64.2, ROW5.8 (Pin_8)
- new net: R54.1, U5.17 (Q2)
- new net: R54.2, ROW4.6 (Pin_6)
- new net: R33.2, ROW2.1 (Pin_1)
- new net: R34.2, ROW2.2 (Pin_2)
- new net: R36.2, ROW2.4 (Pin_4)
- new net: R37.2, ROW2.5 (Pin_5)
- new net: R38.2, ROW2.6 (Pin_6)
- new net: R39.2, ROW2.7 (Pin_7)
- new net: R40.2, ROW2.8 (Pin_8)
- new net: U1.10 (~{Y5}), U7.11 (CP)
- new net: U1.11 (~{Y4}), U6.11 (CP)
- new net: U1.12 (~{Y3}), U5.11 (CP)
- new net: U1.13 (~{Y2}), U4.11 (CP)
- new net: U1.14 (~{Y1}), U3.11 (CP)
- new net: U1.9 (~{Y6}), U8.11 (CP)
- new net: R87.2, ROW8.7 (Pin_7)
- new net: R44.1, U4.15 (Q4)
- new net: R44.2, ROW3.4 (Pin_4)
- new net: R61.1, U6.16 (Q3)
- new net: R67.1, U7.14 (Q5)
- new net: R67.2, ROW6.3 (Pin_3)
- new net: Q3.2 (B), R3.2
- new net: R76.1, U8.15 (Q4)
- new net: R76.2, ROW7.4 (Pin_4)
- new net: R73.2, ROW7.1 (Pin_1)
- new net: R74.2, ROW7.2 (Pin_2)
- new net: R75.2, ROW7.3 (Pin_3)
- new net: R77.2, ROW7.5 (Pin_5)
- new net: R78.2, ROW7.6 (Pin_6)
- new net: R79.2, ROW7.7 (Pin_7)
- new net: R39.1, U3.18 (Q1)
- new net: R83.2, ROW8.3 (Pin_3)
- new net: R88.2, ROW8.8 (Pin_8)
- new net: R53.1, U5.16 (Q3)
- new net: R53.2, ROW4.5 (Pin_5)
- new net: R41.1, U4.12 (Q7)
- new net: R42.1, U4.13 (Q6)
- new net: R43.1, U4.14 (Q5)
- new net: R45.1, U4.16 (Q3)
- new net: R46.1, U4.17 (Q2)
- new net: R48.1, U4.19 (Q0)
- new net: R85.2, ROW8.5 (Pin_5)
- new net: R82.2, ROW8.2 (Pin_2)
- new net: R84.2, ROW8.4 (Pin_4)
- new net: R86.2, ROW8.6 (Pin_6)
- new net: Q7.2 (B), R7.2
- new net: R66.2, ROW6.2 (Pin_2)
- new net: R68.2, ROW6.4 (Pin_4)
- new net: R69.2, ROW6.5 (Pin_5)
- new net: R72.2, ROW6.8 (Pin_8)
- new net: R34.1, U3.13 (Q6)
- new net: R38.1, U3.17 (Q2)
- new net: R62.1, U6.17 (Q2)
- new net: R40.1, U3.19 (Q0)
- new net: R73.1, U8.12 (Q7)
- new net: R55.1, U5.18 (Q1)
- new net: R55.2, ROW4.7 (Pin_7)
- new net: R79.1, U8.18 (Q1)
- new net: R43.2, ROW3.3 (Pin_3)
- new net: R27.2, ROW1.3 (Pin_3)
- new net: R46.2, ROW3.6 (Pin_6)
- new net: R60.1, U6.15 (Q4)
- new net: R78.1, U8.17 (Q2)
- new net: R74.1, U8.13 (Q6)
- new net: R72.1, U7.19 (Q0)
- new net: R25.2, ROW1.1 (Pin_1)
- new net: R69.1, U7.16 (Q3)
- new net: Q2.2 (B), R2.2
- new net: R26.2, ROW1.2 (Pin_2)
- new net: R52.1, U5.15 (Q4)
- new net: R52.2, ROW4.4 (Pin_4)
- new net: R66.1, U7.13 (Q6)
- new net: R68.1, U7.15 (Q4)
- new net: R36.1, U3.15 (Q4)
- new net: R58.1, U6.13 (Q6)
- new net: R37.1, U3.16 (Q3)
- new net: R33.1, U3.12 (Q7)
- new net: Q6.2 (B), R6.2
- new net: R29.2, ROW1.5 (Pin_5)
- new net: R64.1, U6.19 (Q0)
- new net: R41.2, ROW3.1 (Pin_1)
- new net: Q4.2 (B), R4.2
- new net: R31.2, ROW1.7 (Pin_7)
- new net: R77.1, U8.16 (Q3)
- new net: R42.2, ROW3.2 (Pin_2)
- new net: R49.1, U5.12 (Q7)
- new net: R49.2, ROW4.1 (Pin_1)
- new net: R48.2, ROW3.8 (Pin_8)
- new net: R57.1, U6.12 (Q7)
- new net: R45.2, ROW3.5 (Pin_5)
- new net: R50.1, U5.13 (Q6)
- new net: R56.1, U5.19 (Q0)
- new net: R50.2, ROW4.2 (Pin_2)
- new net: R56.2, ROW4.8 (Pin_8)
- new net: R75.1, U8.14 (Q5)
Other:
- moved on the sheet: A1, C1, C10, C11, C12, C2, C3, C4, C5, C6, C7, C8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

Commit message: Update Matrix.kicad_sch
Parts:
- removed A1: Arduino_Nano_v3.x, Module:Arduino_Nano, symbol MCU_Module:Arduino_Nano_v3.x
- added U10: ESP32-S3, Package_DFN_QFN:QFN-56-1EP_7x7mm_P0.4mm_EP4x4mm, symbol MCU_Espressif:ESP32-S3
- C1, C2, C3, C4, C5, C6, C7, C8, C9: value C -> 0.1uf
Connections:
- net A1: now also U10.14 (GPIO9)
- net A2: now also U10.15 (GPIO10)
- net A3: now also U10.16 (GPIO11)
- net D0: now also U10.6 (GPIO1)
- net D1: now also U10.7 (GPIO2)
- net D2: now also U10.8 (GPIO3)
- net D3: now also U10.9 (GPIO4)
- net D4: now also U10.10 (GPIO5)
- net D5: now also U10.11 (GPIO6)
- net D6: now also U10.12 (GPIO7)
- net D7: now also U10.13 (GPIO8)
- net GND: now also U1.8 (GND)
- net OE: now also U10.18 (GPIO13)
- new net: U10.2 (VDD3P3), U10.3 (VDD3P3)
- new net: U10.55 (VDDA), U10.56 (VDDA)
- new net CATHODE1: U10.19 (GPIO14)
- new net CATHODE2: U10.21 (XTAL_32K_P/GPIO15)
- new net CATHODE3: U10.22 (XTAL_32K_N/GPIO16)
- new net CATHODE4: U10.23 (GPIO17)
- new net CATHODE5: U10.24 (GPIO18)
- new net CATHODE6: U10.27 (GPIO21)
- new net CATHODE7: U10.37 (SPICLK_P/GPIO47)
- new net CATHODE8: U10.36 (SPICLK_N/GPIO48)
- new net CLK: U10.17 (GPIO12)
Other:
- moved on the sheet: C1, C10, C11, C12, C2, C3, C4, C5, C6, C7, C8, C9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

Commit message: Update Matrix.kicad_sch
Parts:
- added AE1: Antenna_Chip, symbol Device:Antenna_Chip
- added C13, C24, C25: 10uf, symbol Device:C
- added C14, C22: 1uf, symbol Device:C
- added C15, C16, C17, C18, C19, C20, C21: 0.1uf, symbol Device:C
- added C23: 22uf, symbol Device:C
- added C26: 100nf, symbol Device:C
- added C27, C28: 12pf, symbol Device:C
- added C29, C30, C31, C32: 1.5pf, symbol Device:C
- added D1: SS34, Diode_SMD:D_SMA, symbol Diode:SS34
- added D2: ESD9B3.3ST5G, Diode_SMD:D_SOD-923, symbol Diode:ESD9B3.3ST5G
- added J2: USB_C_Receptacle_USB2.0_16P, symbol Connector:USB_C_Receptacle_USB2.0_16P
- added L1: 2.0nH(0.1nH) 500mA, symbol Device:L
- added L2: 24 nh, symbol Device:L
- added L3: 2.7nh, symbol Device:L
- added L4: 2.2nh, symbol Device:L
- added R89, R90: 5.1k, symbol Device:R
- added U11: AP2112K-3.3, Package_TO_SOT_SMD:SOT-23-5, symbol Regulator_Linear:AP2112K-3.3
- added U13: W25Q32JVSS, Package_SO:SOIC-8_5.3x5.3mm_P1.27mm, symbol Memory_Flash:W25Q32JVSS
- added Y1: 40MHz, symbol Device:Crystal
Connections:
- net +5V: now also C23.1, C24.2, D1.1 (K), U11.1 (VIN), U11.3 (EN)
- net GND: now also U10.57 (GND), AE1.1 (FEED), C13.2, C14.2, C15.2, C16.2, C17.2, C18.2, C19.2, C20.2, C21.2, C22.2, C23.2, C24.1, C25.2, C26.2, C27.1, C28.1, C29.2, C30.2, C31.2, C32.2, D2.1 (A1), J2.A1 (GND), J2.A12 (GND), J2.B1 (GND), J2.B12 (GND), J2.SH (SHIELD), R89.1, R90.1, U11.2 (GND), U13.4 (GND)
- net at U10.1 (LNA_IN): now also C29.1, L3.1
- net at U10.2 (VDD3P3), U10.3 (VDD3P3): now also C15.1, L1.2
- net +3.3V: now reaches U10.20 (VDD3P3_RTC)
- net +3.3V: now also U10.29 (VDD_SPI), U10.46 (VDD3P3_CPU), U10.55 (VDDA), U10.56 (VDDA), C13.1, C14.1, C16.1, C17.1, C18.1, C19.1, C20.1, C21.1, C22.1, C25.1, C26.1, L1.1, U11.5 (VOUT), U13.8 (VCC)
- net D-: now reaches U10.25 (GPIO19/USB_D-)
- net D-: now also J2.A7 (D-), J2.B7 (D-)
- net D+: now reaches U10.26 (GPIO20/USB_D+)
- net D+: now also J2.A6 (D+), J2.B6 (D+)
- net SPIHD: now reaches U10.30 (SPIHD)
- net SPIHD: now also U13.7 (~{HOLD}/~{RESET}/IO_{3})
- net SPICS0: now reaches U10.32 (SPICS0)
- net SPICS0: now also U13.1 (~{CS})
- net SPICLK: now reaches U10.33 (SPICLK)
- net SPICLK: now also U13.6 (CLK)
- net SPIQ: now reaches U10.34 (SPIQ)
- net SPIQ: now also U13.2 (DO/IO_{1})
- net SPID: now reaches U10.35 (SPID)
- net SPID: now also U13.5 (DI/IO_{0})
- net at U10.53 (XTAL_N): now also C28.2, Y1.1
- net at U10.54 (XTAL_P): now also L2.2
- net CLK: no longer names the net of U10.17 (GPIO12)
- new net: J2.B5 (CC2), R90.2
- new net: C27.2, L2.1, Y1.2
- new net: J2.A5 (CC1), R89.2
- new net: C30.1, C31.1, L3.2, L4.1
- new net: D1.2 (A), J2.A4 (VBUS), J2.A9 (VBUS), J2.B4 (VBUS), J2.B9 (VBUS)
- new net: AE1.2 (PCB_Trace), C32.1, D2.2 (A2), L4.2
- new net SPIWP: U13.3 (~{WP}/IO_{2})
- no-connect marks 0 -> 2
Other:
- note added: "FLASH"
- note added: "Power Supply"

Commit message: Update Matrix.kicad_sch
Parts:
- added C33: C, symbol Device:C
- L1: value 2.0nH(0.1nH) 500mA -> 2.0nh(0.1nh) 500mA
- L2: value 24 nh -> 24nh
- Y1: value 40MHz -> 40MHz (+-10ppm)
Connections:
- net +3.3V: now also U1.16 (VCC), U1.6 (E2), U2.20 (VCC), U3.20 (VCC), U4.20 (VCC), U5.20 (VCC), U6.20 (VCC), U7.20 (VCC), U8.20 (VCC), U9.20 (VCC)
- net +5V: no longer U1.4 (~{E0})
- net GND: now also U1.4 (~{E0}); no longer U1.6 (E2), U2.20 (VCC), U3.20 (VCC), U4.20 (VCC), U5.20 (VCC), U6.20 (VCC), U7.20 (VCC), U8.20 (VCC), U9.20 (VCC)
Other:
- note added: "(Near VCC of 74HC574's and 74HC138) 0.1uf x 9"
- note added: "ESP-32 S3"
- moved on the sheet: AE1, C1, C10, C11, C12, C13, C14, C15, C16, C17, C18, C19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

Commit message: Update Matrix.kicad_sch
Parts:
- added U12: ER_OLEDM0.91_1x-I2C, Display:ER_OLEDM0.91_1x-I2C, symbol Display_Graphic:ER_OLEDM0.91_1x-I2C
Connections:
- net +3.3V: now also U12.2 (VCC)
- net GND: now also U12.1 (GND)
- net SDA: now reaches U10.40 (GPIO35)
- net SDA: now also U12.4 (SDA)
- net SCL: now reaches U10.41 (GPIO36)
- net SCL: now also U12.3 (SCL)
Other:
- note added: "OLED display"
- moved on the sheet: AE1, C13, C14, C15, C16, C17, C18, C19, C20, C21, C22, C27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

Commit message: Update Matrix.kicad_sch
Parts:
- removed C33: C, symbol Device:C
- AE1: footprint (none) -> AH316M245001-T:ANTC3216X60N
- C13, C14, C15, C16, C17, C18, C19, C20, C21, C22, C23, C24, C25, C26, C27, C28, C29, C30, C31, C32: footprint (none) -> Capacitor_SMD:C_0805_2012Metric_Pad1.18x1.45mm_HandSolder
- J2: footprint (none) -> Connector_USB:USB_C_Receptacle_GCT_USB4105-xx-A_16P_TopMnt_Horizontal
- L1, L2, L3, L4: footprint (none) -> Inductor_SMD:L_0805_2012Metric_Pad1.05x1.20mm_HandSolder
- R89, R90: footprint (none) -> Resistor_SMD:R_0805_2012Metric_Pad1.20x1.40mm_HandSolder
- Y1: footprint (none) -> Crystal:Crystal_SMD_3225-4Pin_3.2x2.5mm_HandSoldering
Connections:
- net CATHODE1 is gone; now on net CATHODE 1: U10.19 (GPIO14)
- net CATHODE2 is gone; now on net CATHODE 2: U10.21 (XTAL_32K_P/GPIO15)
- net CATHODE3 is gone; now on net CATHODE 3: U10.22 (XTAL_32K_N/GPIO16)
- net CATHODE4 is gone; now on net CATHODE 4: U10.23 (GPIO17)
- net CATHODE5 is gone; now on net CATHODE 5: U10.24 (GPIO18)
- net CATHODE6 is gone; now on net CATHODE 6: U10.27 (GPIO21)
- net CATHODE7 is gone; now on net CATHODE 7: U10.37 (SPICLK_P/GPIO47)
- net CATHODE8 is gone; now on net CATHODE 8: U10.36 (SPICLK_N/GPIO48)
- net GND: now also AE1.2 (PCB_Trace); no longer AE1.1 (FEED)
- net SPIWP: now also U10.31 (SPIWP)
- net at C32.1, D2.2 (A2), L4.2: now also AE1.1 (FEED); no longer AE1.2 (PCB_Trace)
- no-connect marks 2 -> 18
Other:
- moved on the sheet: AE1, C24
