File: Matrix/Matrix.kicad_sch (KiCad schematic)
At the start: 169 parts, among them J1 Conn_01x08, J2 USB_C_Receptacle_USB2.0_16P, Q1 2N2219, Q10 2N2219, Q11 2N2219, Q12 2N2219, Q13 2N2219, Q14 2N2219, Q15 2N2219, Q16 2N2219, Q2 2N2219, Q3 2N2219, Q4 2N2219, Q5 2N2219, Q6 2N2219, Q7 2N2219, Q8 2N2219, Q9 2N2219, U1 74HC138, U10 ESP32-S3, U11 AP2112K-3.3, U12 ER_OLEDM0.91_1x-I2C, U13 W25Q32JVSS, U2 74HC574N, U3 74HC574N, U4 74HC574N, U5 74HC574N, U6 74HC574N, U7 74HC574N, U8 74HC574N, U9 74HC574N, Y1 40MHz (+-10ppm)

Commit message: Update Matrix.kicad_sch
Connections:
- net +3.3V: now also C1.1, C2.1, C3.1, C4.1, C5.1, C6.1, C7.1, C8.1, C9.1
- net +5V: no longer C1.1, C2.1, C3.1, C4.1, C5.1, C6.1, C7.1, C8.1, C9.1
Other:
- moved on the sheet: C1, C2, C3, C4, C5, C6, C7, C8, C9, U12
